File: BuzzWireGame/BuzzWireGame.kicad_pcb (KiCad board)
At the start: 2 copper layers, 0 parts

Commit message: Finish schm and PCB design for v1.0
Parts:
- added BT1: 9V Battery, TerminalBlock:TerminalBlock_bornier-2_P5.08mm, F.Cu at (135.1, 64.8)
- added C1: 10nF, Capacitor_SMD:C_1206_3216Metric, F.Cu at (150.7, 98.8)
- added C2: 1uF, Capacitor_SMD:C_1206_3216Metric, F.Cu at (142.8, 73.0)
- added C3: 100n, Capacitor_SMD:C_1206_3216Metric, F.Cu at (141.0, 88.8)
- added C4: 10nF, Capacitor_SMD:C_1206_3216Metric, F.Cu at (123.5, 99.4)
- added C5: 4.7uF, Capacitor_THT:CP_Radial_D4.0mm_P2.00mm, F.Cu at (117.8, 99.4)
- added D1: RED, LED_THT:LED_D5.0mm_Clear, F.Cu at (176.1, 107.0)
- added D2: RED, LED_THT:LED_D5.0mm_Clear, F.Cu at (109.4, 93.2)
- added D3: GREEN, LED_THT:LED_D5.0mm_Clear, F.Cu at (178.8, 92.0)
- added G***: LOGO, MyFootprintLibrary:eestec_ns_logo, F.Cu at (122.8, 111.5)
- added G***: LOGO, MyFootprintLibrary:konteh_logo, B.Cu at (160.2, 64.5)
- added H1: Hole, MountingHole:MountingHole_3.2mm_M3_Pad_Via, F.Cu at (105.0, 65.0)
- added H2: Hole, MountingHole:MountingHole_3.2mm_M3_Pad_Via, F.Cu at (185.0, 65.0)
- added H3: Hole, MountingHole:MountingHole_3.2mm_M3_Pad_Via, F.Cu at (105.0, 115.0)
- added H4: Hole, MountingHole:MountingHole_3.2mm_M3_Pad_Via, F.Cu at (185.0, 115.0)
- added J1: Barrel_Jack_Switch, Connector_BarrelJack:BarrelJack_Horizontal, F.Cu at (119.0, 74.8)
- added J2: Wire track terminal, TerminalBlock:TerminalBlock_bornier-2_P5.08mm, F.Cu at (185.8, 77.8)
- added LS1: Piezo buzzer, Buzzer_Beeper:Indicator_PUI_AI-1440-TWT-24V-2-R, F.Cu at (149.5, 71.5)
- added Q1: BC549, Package_TO_SOT_THT:TO-92_Inline, F.Cu at (169.8, 93.5)
- added Q2: BC549, Package_TO_SOT_THT:TO-92_Inline, F.Cu at (169.6, 108.0)
- added R1: 1kΩ, Resistor_THT:R_Axial_DIN0207_L6.3mm_D2.5mm_P10.16mm_Horizontal, F.Cu at (160.8, 87.7)
- added R10: 22Ω, Resistor_THT:R_Axial_DIN0207_L6.3mm_D2.5mm_P10.16mm_Horizontal, F.Cu at (179.4, 101.0)
- added R11: 180kΩ, Resistor_THT:R_Axial_DIN0207_L6.3mm_D2.5mm_P10.16mm_Horizontal, F.Cu at (129.2, 93.2)
- added R12: 220Ω, Resistor_THT:R_Axial_DIN0207_L6.3mm_D2.5mm_P10.16mm_Horizontal, F.Cu at (109.4, 97.5)
- added R2: 100Ω, Resistor_THT:R_Axial_DIN0207_L6.3mm_D2.5mm_P10.16mm_Horizontal, F.Cu at (175.8, 75.0)
- added R3: 100Ω, Resistor_THT:R_Axial_DIN0207_L6.3mm_D2.5mm_P10.16mm_Horizontal, F.Cu at (175.8, 69.8)
- added R4: 2.2kΩ, Resistor_THT:R_Axial_DIN0207_L6.3mm_D2.5mm_P10.16mm_Horizontal, F.Cu at (154.1, 82.0)
- added R5: 4.7kΩ, Resistor_THT:R_Axial_DIN0207_L6.3mm_D2.5mm_P10.16mm_Horizontal, F.Cu at (165.7, 80.5)
- added R6: 100Ω, Resistor_THT:R_Axial_DIN0207_L6.3mm_D2.5mm_P10.16mm_Horizontal, F.Cu at (186.0, 98.7)
- added R7: 4k7Ω, Resistor_THT:R_Axial_DIN0207_L6.3mm_D2.5mm_P10.16mm_Horizontal, F.Cu at (186.0, 96.0)
- added R8: 1kΩ, Resistor_THT:R_Axial_DIN0207_L6.3mm_D2.5mm_P10.16mm_Horizontal, F.Cu at (129.2, 78.4)
- added R9: 22Ω, Resistor_THT:R_Axial_DIN0207_L6.3mm_D2.5mm_P10.16mm_Horizontal, F.Cu at (169.4, 86.2)
- added RV1: 1kΩ, Potentiometer_THT:Potentiometer_Alps_RK163_Single_Horizontal, F.Cu at (149.5, 113.0)
- added SW1: SW_Push, Button_Switch_THT:SW_PUSH_6mm_H4.3mm, F.Cu at (135.5, 114.3)
- added U1: NE555P, Package_DIP:DIP-8_W7.62mm, F.Cu at (145.2, 87.7)
- added U2: NE555P, Package_DIP:DIP-8_W7.62mm, F.Cu at (116.2, 85.6)
Routing:
- net +9V: track 0.00 -> 172.7 mm
- net TIMER_RESET: track 0.00 -> 109.8 mm
- net Net-(J2-Pin_2): track 0.00 -> 78.0 mm
- net Net-(U1-DIS): track 0.00 -> 41.9 mm
- net Net-(U2-THR): track 0.00 -> 33.1 mm
- net Net-(U1-Q): track 0.00 -> 25.2 mm
- net Net-(U1-THR): track 0.00 -> 24.3 mm
- net Net-(D3-A): track 0.00 -> 19.4 mm
- net BATT_NEG: track 0.00 -> 18.6 mm
- net Net-(R1-Pad2): track 0.00 -> 15.7 mm
- net Net-(U2-DIS): track 0.00 -> 10.2 mm
- net Net-(LS1-Pad2): track 0.00 -> 9.29 mm
- net Net-(D1-A): track 0.00 -> 8.16 mm
- net Net-(D1-K): track 0.00 -> 6.89 mm
- net Net-(D2-A): track 0.00 -> 6.83 mm
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- added copper zone on B.Cu, net GND
- added copper zone on F.Cu, net GND
Other:
- board outline added: 90 x 60 mm
- board text added: "+"
- board text added: "- +"
- board text added: "100nF"
- board text added: "100Ω"
- board text added: "10nF"
- board text added: "180kΩ"
- board text added: "1kΩ"
- board text added: "1uF"
- board text added: "2.2kΩ"
- board text added: "220Ω"
- board text added: "22Ω"
- board text added: "4.7kΩ"
- board text added: "4.7uF"
- board text added: "9V BATT"
- board text added: "9V DC"
- board text added: "BC549"
- board text added: "GREEN"
- board text added: "JLCJLCJLCJLC"
- board text added: "NE555"
- board text added: "ON"
- board text added: "PIEZO BUZZER"
- board text added: "RED"
- board text added: "TEST"
- board text added: "TONE"
- board text added: "WIRES"
- board text added: "v1.0"
- board text added: "www.github.com/AleksaHeler/EESTEC-Buzz-Wire-Game"
